Commit message: cleaned up config, launch and quadrotor urdf files

File: world/quadrotor_urdf/uav2.gazebo.xacro (robot description, xacro)
@@ -2,5 +2,5 @@
 <robot name="quadrotor"
     xmlns:xacro="http://www.ros.org/wiki/xacro">
-    <xacro:include filename="$(find aro)/world/quadrotor_urdf/quadrotor.urdf.xacro" />
+    <xacro:include filename="$(find aro)/world/quadrotor_urdf/uav2.urdf.xacro" />
     <xacro:include filename="$(find hector_quadrotor_gazebo)/urdf/quadrotor_plugins.gazebo.xacro" />
 </robot>

File: world/quadrotor_urdf/uav2.urdf.xacro (robot description, xacro)
@@ -3,5 +3,5 @@
   xmlns:xacro="http://www.ros.org/wiki/xacro">
   <!-- Included URDF Files -->
-  <xacro:include filename="$(find aro)/world/quadrotor_urdf/quadrotor_base.urdf.xacro" />
+  <xacro:include filename="$(find aro)/world/quadrotor_urdf/uav2_base.urdf.xacro" />
   <!-- Instantiate quadrotor_base_macro once (has no parameters atm) -->
   <xacro:quadrotor_base_macro />

File: world/quadrotor_urdf/uav2_base.urdf.xacro (robot description, xacro)
@@ -1,5 +1,4 @@
 <?xml version="1.0"?>
 <robot xmlns:xacro="http://www.ros.org/wiki/xacro">
-  <xacro:include filename="$(find hector_sensors_description)/urdf/sonar_sensor.urdf.xacro" />
   <xacro:property name="pi" value="3.1415926535897931" />
   <!-- Main quadrotor link -->
@@ -24,8 +23,4 @@
       </collision>
     </link>
-    <!-- Sonar height sensor -->
-    <xacro:sonar_sensor name="sonar" parent="base_link" ros_topic="sonar_height" update_rate="30" min_range="0.03" max_range="3.0" field_of_view="${5*pi/180}" ray_count="10">
-      <origin xyz="0.0 0.0 -0.12" rpy="0 ${90*pi/180} 0"/>
-    </xacro:sonar_sensor>
   </xacro:macro>
 </robot>
